Commit message: Updated to add empty room and allow launch in empty room

File: src/walker/resource/my_robot.urdf (robot description, URDF)
Before this commit: robot Myrobot, 0 links, 0 joints
Links:
- added link base_link
- added link ds0_link
- added link ds1_link
Joints:
- added joint ds0_joint: type fixed, parent base_link, child ds0_link, origin xyz=0.042 0.02 0.063 rpy=0 0 0.5236
- added joint ds1_joint: type fixed, parent base_link, child ds1_link, origin xyz=0.042 -0.02 0.063 rpy=0 0 -0.5236
